File: HW/ControllerStage.sch (KiCad schematic (older format))
At the start: 39 parts, among them J1 Load_relay, J10 Trigger BTN, J11 External trigger, J2 Mosfet_temp, J3 Load_relay, J6 reset, J8 Encoder and LCD interface, J9 ScopeTest, Q1 BC847, Q2 BC847, Q4 BUZ11, Q5 BUZ11, U1 SN74LVC1G14, U16 PC817, U22 SN74LVC1G14, U23 DS3231, U6 BluePill_STM32F103C, U7 MCP4725, U9 LM75

Commit message: cleanup - getting ready for v0.2
Connections:
- net encA: now also U6.30 (PA15); no longer U6.32 (PB4)
- net loadOff: no longer names the net of U6.29 (PA12_USBD+)
Other:
- note added: "FEL footprint"
Changed lines of the file:
@@
 Text GLabel 9300 4800 2    60   Input ~ 0
 encB
-Text GLabel 9300 4700 2    60   Input ~ 0
+Text GLabel 9300 4900 2    60   Input ~ 0
 encA
 $Comp
@@
 Text Notes 900  6250 0    60   ~ 0
 14 bits = 4096 steps\n1 step=1mV\n1mV@0.1 Ohm = 10mA \n40AMAX
-Text GLabel 9300 5000 2    60   Input ~ 0
-loadOff
 $Comp
 L PC817 U16
@@
 Connection ~ 2700 10400
 Connection ~ 2700 10300
+Text Notes 15000 3100 0    60   ~ 0
+FEL footprint
+Text Notes 15050 4650 0    60   ~ 0
+FEL footprint
+Text Notes 2800 9950 0    60   ~ 0
+FEL footprint
 $EndSCHEMATC
