File: HW/file59D92098.sch (KiCad schematic (older format))
At the start: 36 parts, among them J4 BARREL_JACK, U10 LT1054, U2 INA219, U21 LM321, U3 lm2931-5.0, U4 LM317_3PinPackage, U8 MAX6241

Commit message: söndags
Parts:
- U21: symbol LM321 -> LM321-RESCUE-ControllerStage
Changed lines of the file:
@@
 LIBS:contrib
 LIBS:valves
-LIBS:Peters
-LIBS:bluepill_breakouts
 LIBS:SN74LVC1G14DBVT
 LIBS:ControllerStage-cache
@@
 $EndComp
 $Comp
-L LM321 U21
+L LM321-RESCUE-ControllerStage U21
 U 1 1 5ABF4E5A
 P 9650 2200
+AR Path="/5ABF4E5A" Ref="U21"  Part="1"
+AR Path="/59D92099/5ABF4E5A" Ref="U21"  Part="1"
 F 0 "U21" H 9650 2500 50  0000 L CNN
 F 1 "LM321" H 9650 2400 50  0000 L CNN
