File: HW/file5A104BBF.sch (KiCad schematic (older format))
At the start: 53 parts, among them J12 Remote_sense, J5 Dut+, J7 DUT-, Q3 STW45NM50, U11 LM321, U12 LM35, U13 ADS1115, U14 OP07, U15 OP07, U17 OP07, U18 OP07, U19 LM321, U20 TL431A

Commit message: söndags
Parts:
- U11, U19: symbol LM321 -> LM321-RESCUE-ControllerStage
Changed lines of the file:
@@
 LIBS:contrib
 LIBS:valves
-LIBS:Peters
-LIBS:bluepill_breakouts
 LIBS:SN74LVC1G14DBVT
 LIBS:ControllerStage-cache
@@
 $EndComp
 $Comp
-L LM321 U11
+L LM321-RESCUE-ControllerStage U11
 U 1 1 5A105281
 P 9200 5000
+AR Path="/5A105281" Ref="U11"  Part="1"
+AR Path="/5A104BC0/5A105281" Ref="U11"  Part="1"
 F 0 "U11" H 9200 5300 50  0000 L CNN
 F 1 "LM321" H 9200 5200 50  0000 L CNN
@@
 	2000 5850 2200 5850
 $Comp
-L LM321 U19
+L LM321-RESCUE-ControllerStage U19
 U 1 1 5ABE9BAF
 P 1300 5500
+AR Path="/5ABE9BAF" Ref="U19"  Part="1"
+AR Path="/5A104BC0/5ABE9BAF" Ref="U19"  Part="1"
 F 0 "U19" H 1300 5800 50  0000 L CNN
 F 1 "LM321" H 1300 5700 50  0000 L CNN

Commit message: cleanup - getting ready for v0.2
Parts:
- removed C22, C23: 0.1u, Capacitors_SMD:C_0805_HandSoldering, symbol C
- removed R44: 4M7, Resistors_SMD:R_0805_HandSoldering, symbol R
- removed U14: OP07, Housings_DIP:DIP-8_W7.62mm_Socket_LongPads, symbol OP07
- removed U19: LM321, TO_SOT_Packages_SMD:SOT-23-5_HandSoldering, symbol LM321-RESCUE-ControllerStage
- added R? (x2): 1M, Resistors_SMD:R_0805_HandSoldering, symbol R
- added R?: 100R, Resistors_SMD:R_0805_HandSoldering, symbol R
Connections:
- net +12V: now also RV3.2, U15.4 (V-)
- net +5V: now also RV2.2
- net -5V: no longer RV2.2, RV3.2, U15.4 (V-)
- net Earth: now also R?.1, R?.2
- net at Q3.1 (G), R28.1: now also R?.1; no longer C29.1, U15.6
- net at C21.1, R21.1, U13.6 (AIN2): now also R35.2; no longer R35.1
- net at R26.2, R36.2, U18.6: now also R35.1
- net at R36.1, R40.2, U18.2 (-): now also R?.1
- net at R37.2, R41.2, U18.3 (+): now also R?.2
- new net: C29.1, R?.2, U15.6
Other:
- note removed: "Goes +3v3 to force output LOW"
- moved on the sheet: R28, R35, R37
