File: HW/v2/v2.kicad_pcb (KiCad board)
At the start: 2 copper layers, 142 parts, among them J1 Encoder and LCD interface, J10 RST, J11 ScopeTest, J12 Trigger BTN, J13 External trigger, J14 Barrel_Jack, J2 Fan_conn, J3 SDcardHeader, J4 OUT2, J5 OUT2, J6 DUT+, J7 DUT-, J8 Remote_sense, J9 GPIO, Q1 BC847, Q2 BC847, Q3 IRF7341, Q4 STW45NM50, U1 LM75, U10 Temp amp, U11 LM35, U12 Bluepill, U13 DS3231 RTC, U14 TRIG, U15 SN74LVC2G14, U16 PC817, U17 LT1054 neg5v, U18 INA219, U19 LM7805, U2 TL431A, U20 LM1117-3.3, U21 Vref, U22 AD8628, U23 LM321, U3 ADS1115, U4 Gate DRV, U5 Volt buffer, U6 Current amp, U7 Volt sense, U8 MCP4725, U9 AD8628

Commit message: layout
Parts:
- added R112: 10K, Resistors_SMD:R_0805_HandSoldering, F.Cu at (204.3, 117.7)
- C12, C7, D3, R23, R24, R6, R8, U22, U9: moved to B.Cu
- Q4: footprint TO_SOT_Packages_THT:TO-247_TO-3P_Vertical -> Load_mosfet
- R13: footprint Resistors_THT:R_Axial_DIN0516_L15.5mm_D5.0mm_P20.32mm_Horizontal -> Loadresistor
- moved J6 394.7 mm to (244.4, 133.5), turned to 90 degrees
- moved F1 390.8 mm to (231.4, 133.3), turned to 180 degrees
- moved U5 377.9 mm to (272.1, 50.7)
- moved U3 374.5 mm to (239.0, 26.9)
- moved J7 368.8 mm to (243.5, 115.8), turned to 90 degrees
- moved R13 362.5 mm to (229.6, 116.5)
- moved Q4 361.5 mm to (208.6, 113.3), turned to 270 degrees
- moved RV4 351.5 mm to (260.9, 46.9)
- moved U7 351.3 mm to (259.3, 50.9)
- moved D3 349.4 mm to (221.0, 124.3)
- moved R14 324.5 mm to (254.2, 54.2), turned to 90 degrees
- moved U6 316.6 mm to (219.9, 96.6), turned to 270 degrees
- moved U9 314.7 mm to (193.7, 130.5), turned to 180 degrees
- moved C14 312.4 mm to (214.8, 92.1)
- moved C10 299.5 mm to (192.8, 106.0), turned to 180 degrees
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Connections:
- C7 pad 2: (no net) -> -5V
- U4 pad 4: +12V -> -5V
- U9 pad 7: 4.096V -> +5V
Routing:
- net +12V: track 0.00 -> 52.0 mm
- net 4.096V: track 0.00 -> 35.3 mm, vias 0 -> 1
- net Net-(Q4-Pad2): track 0.00 -> 32.8 mm
- net Earth: track 0.00 -> 23.7 mm
- net Net-(RV6-Pad3): track 0.00 -> 17.3 mm, vias 0 -> 1
- net CurrentSet: track 0.00 -> 12.5 mm
- net Net-(Q4-Pad1): track 0.00 -> 12.4 mm
- net Net-(R22-Pad1): track 0.00 -> 10.3 mm, vias 0 -> 1
- net Net-(R23-Pad2): track 0.00 -> 9.72 mm
- net Net-(R5-Pad2): track 0.00 -> 8.63 mm
- net Net-(RV6-Pad2): track 0.00 -> 8.59 mm, vias 0 -> 1
- net Net-(D3-Pad1): track 0.00 -> 8.55 mm
- net Net-(R24-Pad2): track 0.00 -> 8.25 mm
- net Net-(C12-Pad1): track 0.00 -> 7.52 mm
- net -5V: track 0.00 -> 5.15 mm
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- added copper zone on B.Cu, net /Mosfet stage/Dut+_efter_säkring
- added copper zone on F.Cu, net /Mosfet stage/Dut+_efter_säkring
- added copper zone on B.Cu, net Earth
- added copper zone on F.Cu, net Earth
- added copper zone on B.Cu, net Net-(D3-Pad1)
- added copper zone on F.Cu, net Net-(D3-Pad1)

Commit message: layout
Parts:
- added C16: C, Capacitors_SMD:C_0805_HandSoldering, F.Cu at (230.9, 78.1)
- C14, C42, C8, R11, R17, R18, R19, R20, R21, R7, R9, U23: moved to B.Cu
- moved U11 200.6 mm to (249.6, 80.0), turned to 270 degrees
- moved U10 198.0 mm to (244.9, 82.7), turned to 270 degrees
- moved D9 162.3 mm to (220.5, -56.1)
- moved R38 162.3 mm to (226.7, -56.0)
- moved J8 160.2 mm to (251.2, 99.3), turned to 270 degrees
- moved C17 150.4 mm to (236.4, 105.4), turned to 180 degrees
- moved R17 147.4 mm to (244.0, 104.3), turned to 90 degrees
- moved C19 139.9 mm to (249.5, 75.8), turned to 90 degrees
- moved R19 139.7 mm to (241.6, 104.3), turned to 90 degrees
- moved R15 138.8 mm to (240.0, 92.0), turned to 180 degrees
- moved RV3 134.4 mm to (206.9, 101.6), turned to 180 degrees
- moved R21 133.3 mm to (245.4, 100.5), turned to 180 degrees
- moved R18 132.3 mm to (244.2, 91.0), turned to 90 degrees
- moved R20 129.0 mm to (245.6, 95.3), turned to 180 degrees
- moved R25 128.5 mm to (241.7, 83.3), turned to 90 degrees
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Routing:
- net +5V: track 0.00 -> 155.0 mm
- net Earth: track 23.7 -> 76.0 mm
- net Net-(R16-Pad1): track 0.00 -> 29.8 mm
- net Curr: track 0.00 -> 28.4 mm
- net -5V: track 5.15 -> 26.3 mm
- net Net-(R15-Pad2): track 0.00 -> 20.5 mm
- net Net-(R11-Pad1): track 0.00 -> 20.3 mm
- net Net-(R17-Pad2): track 0.00 -> 16.9 mm
- net Net-(D9-Pad2): track 0.00 -> 10.1 mm
- net Net-(R14-Pad2): track 0.00 -> 9.75 mm
- net Net-(C11-Pad1): track 0.00 -> 8.68 mm
- net Net-(Q4-Pad2): track 32.8 -> 41.3 mm
- net Net-(RV4-Pad1): track 0.00 -> 7.66 mm
- net Net-(RV4-Pad3): track 0.00 -> 7.62 mm
- net 4.096V: track 35.3 -> 41.1 mm
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
Commit message: friday layout
Parts:
- added REF**: MountingHole_3.2mm_M3, Mounting_Holes:MountingHole_3.2mm_M3, F.Cu at (220.7, 115.6)
- added REF**: MountingHole_3.2mm_M3, Mounting_Holes:MountingHole_3.2mm_M3, F.Cu at (249.2, 45.5)
- added REF**: MountingHole_3.2mm_M3, Mounting_Holes:MountingHole_3.2mm_M3, F.Cu at (160.8, 45.5)
- added REF**: MountingHole_3.2mm_M3, Mounting_Holes:MountingHole_3.2mm_M3, F.Cu at (161.0, 137.9)
- added REF**: JUMPER 5MM, Libs:JUMPER_5MM, F.Cu at (206.0, 72.6)
- C24, C25, C26, C27, C31, C35, L1, R31, R32, R33, U1, U18: moved to B.Cu
- C30: footprint Capacitors_SMD:C_0805_HandSoldering -> Capacitors_Tantalum_SMD:CP_Tantalum_Case-E_EIA-7260-38_Hand
- moved C1 343.4 mm to (-4.97, -79.3)
- moved C2 343.4 mm to (12.2, -104.6)
- moved C3 343.4 mm to (8.71, -90.1)
- moved C4 343.4 mm to (0.18, -79.3)
- moved D2 343.4 mm to (-4.56, -85.8)
- moved J1 343.4 mm to (-22.6, -105.6)
- moved J3 343.4 mm to (-6.60, -105.6)
- moved J4 343.4 mm to (20.2, -105.6)
- moved J5 343.4 mm to (-15.8, -83.5)
- moved Q1 343.4 mm to (-10.6, -78.6)
- moved Q3 343.4 mm to (7.04, -81.0)
- moved R1 343.4 mm to (25.2, -99.0)
- moved R2 343.4 mm to (25.2, -93.3)
- moved R3 343.4 mm to (17.1, -87.5)
- moved R4 343.4 mm to (25.2, -87.6)
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Routing:
- net -5V: track 26.3 -> 259.8 mm
- net +12V: track 52.0 -> 276.9 mm, vias 0 -> 1
- net SCL: track 0.00 -> 198.4 mm, vias 0 -> 1
- net SDA: track 0.00 -> 192.8 mm, vias 0 -> 1
- net +5V: track 155.0 -> 272.2 mm
- net Earth: track 76.0 -> 188.2 mm
- net +3V3: track 0.00 -> 76.0 mm, vias 0 -> 2
- net Net-(C24-Pad1): track 0.00 -> 24.7 mm
- net Net-(C31-Pad1): track 0.00 -> 19.1 mm
- net Net-(C27-Pad1): track 0.00 -> 18.8 mm
- net Net-(C39-Pad1): track 0.00 -> 14.8 mm
- net Net-(R25-Pad1): track 0.00 -> 8.58 mm
- net LoadBlockTemp: track 0.00 -> 5.88 mm
- net Net-(C23-Pad2): track 0.00 -> 5.56 mm
- net Net-(C23-Pad1): track 0.00 -> 5.23 mm
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Other:
- board outline added: 97 x 99.8 mm
- net class Default: clearance 0.3 -> 0.25
- net class power: clearance 0.3 -> 0.4
- rule trace_clearance: 0.3 -> 0.25

Commit message: yup
Parts:
- C28, R27: moved to B.Cu
- moved J2 251.6 mm to (162.6, 88.6), turned to 180 degrees
- moved J3 248.3 mm to (162.6, 76.2), turned to 180 degrees
- moved J1 245.0 mm to (170.7, 45.0), turned to 90 degrees
- moved C4 221.4 mm to (159.3, 74.7), turned to 90 degrees
- moved Q1 218.7 mm to (164.1, 53.1)
- moved U16 217.0 mm to (202.4, 48.0), turned to 270 degrees
- moved U13 213.7 mm to (194.1, 67.1)
- moved J13 206.3 mm to (192.5, 47.8), turned to 180 degrees
- moved J11 202.2 mm to (196.1, 43.9)
- moved J10 201.1 mm to (165.9, 91.7)
- moved D4 201.1 mm to (199.4, 44.2)
- moved J12 196.2 mm to (193.0, 51.1), turned to 180 degrees
- moved Q3 183.9 mm to (71.6, 91.2)
- moved R27 183.5 mm to (182.1, 57.1), turned to 270 degrees
- moved D2 169.4 mm to (67.3, 67.6)
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Connections:
- U12 pad 30: encBTN -> encB
- U12 pad 32: encB -> encBTN
Routing:
- net SDA: track 192.8 -> 278.7 mm, vias 1 -> 2
- net SCL: track 198.4 -> 280.8 mm, vias 1 -> 2
- net encB: track 0.00 -> 38.7 mm
- net encA: track 0.00 -> 35.6 mm
- net encBTN: track 0.00 -> 34.1 mm
- net MOSI: track 0.00 -> 19.5 mm
- net SS: track 0.00 -> 15.5 mm
- net SCK: track 0.00 -> 14.9 mm
- net +12V: track 276.9 -> 291.0 mm
- net Net-(BT1-Pad1): track 0.00 -> 14.1 mm, vias 0 -> 1
- net MISO: track 0.00 -> 11.9 mm
- net +3V3: track 76.0 -> 85.2 mm, vias 2 -> 1
- net fan_PWM: track 0.00 -> 8.24 mm
- net (no net): track 0.00 -> 5.15 mm
- net -5V: track 259.8 -> 260.9 mm
Other:
- board size 97 x 99.8 mm -> 98.3 x 100.8 mm
