File: HW/v2/v2.kicad_pcb (KiCad board)
At the start: 2 copper layers, 97 x 99.8 mm, 149 parts, among them J1 Encoder and LCD interface, J10 RST, J11 ScopeTest, J12 Trigger BTN, J13 External trigger, J14 Barrel_Jack, J2 Fan_conn, J3 SDcardHeader, J4 OUT2, J5 OUT2, J6 DUT+, J7 DUT-, J8 Remote_sense, J9 GPIO, Q1 BC847, Q2 BC847, Q3 IRF7341, Q4 STW45NM50, U1 LM75, U10 Temp amp, U11 LM35, U12 Bluepill, U13 DS3231 RTC, U14 TRIG, U15 SN74LVC2G14, U16 PC817, U17 LT1054 neg5v, U18 INA219, U19 LM7805, U2 TL431A, U20 LM1117-3.3, U21 Vref, U22 AD8628, U23 LM321, U3 ADS1115, U4 Gate DRV, U5 Volt buffer, U6 Current amp, U7 Volt sense, U8 MCP4725, U9 AD8628

Commit message: i2c pots for calibrating
Parts:
- removed the C16 at (230.9, 78.1)
- removed the C16 at (225.0, 89.1)
- removed R112: 10K, Resistors_SMD:R_0805_HandSoldering
- removed REF** (x4): MountingHole_3.2mm_M3, Mounting_Holes:MountingHole_3.2mm_M3
- removed REF**: JUMPER 5MM, Libs:JUMPER_5MM
- removed RV5: 5K, Potentiometers:Potentiometer_Trimmer_ACP_CA9h2.5_Vertical_Px2.5mm_Py5.0mm
- removed RV6: 10K, Potentiometers:Potentiometer_Trimmer_ACP_CA9h2.5_Vertical_Px2.5mm_Py5.0mm
- added C16: C, Capacitors_SMD:C_0805_HandSoldering, B.Cu at (209.6, 92.5)
- added C43: 0.1u, Capacitors_SMD:C_0805_HandSoldering, F.Cu at (148.8, 117.1)
- added J15: Barrel_Jack, Connectors:BARREL_JACK, F.Cu at (369.5, 1.85)
- added R-shunt1: 0.1, LoadResistor:Loadresistor, F.Cu at (208.2, 120.7)
- added R39: 2k7, Resistors_SMD:R_0805_HandSoldering, F.Cu at (394.1, 36.8)
- added U24: Vref, Housings_SOIC:SOIC-8_3.9x4.9mm_Pitch1.27mm, B.Cu at (149.6, 132.3)
- added U25: AD8628, Housings_SOIC:SOIC-8_3.9x4.9mm_Pitch1.27mm, B.Cu at (156.0, 132.3)
- BT1: footprint Battery_Holders:Keystone_3008_1x2450-CoinCell -> Libs:JUMPER_5MM
- C1: moved to B.Cu
- C10: value 10u -> 0.1u; footprint Capacitors_Tantalum_SMD:CP_Tantalum_Case-B_EIA-3528-21_Hand -> Capacitors_SMD:C_0805_HandSoldering; moved to B.Cu
- C11: value 0.1u -> 1n; moved to B.Cu
- C12: value 1n -> 0.1u; moved to F.Cu
- C24, C25, C26, C27, C31, C42, C7, L1, R19, R20, U23: moved to F.Cu
- C30: footprint Capacitors_Tantalum_SMD:CP_Tantalum_Case-E_EIA-7260-38_Hand -> Capacitors_SMD:C_0805_HandSoldering
- C33: value 220u -> 10u; footprint Capacitors_Tantalum_SMD:CP_Tantalum_Case-C_EIA-6032-28_Hand -> Capacitors_SMD:C_0805_HandSoldering
- C34: value 2.2uF -> 100nF
- C35: value 100nF -> 10u; moved to F.Cu
- C36: value 10u -> 100u; footprint Capacitors_SMD:C_0805_HandSoldering -> Capacitors_Tantalum_SMD:CP_Tantalum_Case-C_EIA-6032-28_Hand
- C37: value 100n -> 22u
- C38: value 1uF -> 220u; footprint Capacitors_SMD:C_0805_HandSoldering -> Capacitors_Tantalum_SMD:CP_Tantalum_Case-C_EIA-6032-28_Hand; moved to B.Cu
- C39: value 10u -> 2.2uF; moved to B.Cu
- C40: value 100u -> 100n; footprint Capacitors_Tantalum_SMD:CP_Tantalum_Case-C_EIA-6032-28_Hand -> Capacitors_SMD:C_0805_HandSoldering; moved to B.Cu
- C41: value 22u -> 1uF; moved to B.Cu
- C9: value 0.1u -> 10u; footprint Capacitors_SMD:C_0805_HandSoldering -> Capacitors_Tantalum_SMD:CP_Tantalum_Case-B_EIA-3528-21_Hand; moved to B.Cu
- J1: value Encoder and LCD interface -> Fan_conn; footprint Pin_Headers:Pin_Header_Straight_1x07_Pitch2.54mm -> Pin_Headers:Pin_Header_Straight_1x04_Pitch2.54mm
- J10: value RST -> GPIO
- J11: value ScopeTest -> RST; footprint Libs:JUMPER_5MM -> Pin_Headers:Pin_Header_Straight_1x02_Pitch2.54mm
- J12: value Trigger BTN -> ScopeTest
- J13: value External trigger -> Trigger BTN
- J14: value Barrel_Jack -> External trigger; footprint Connectors:BARREL_JACK -> Libs:JUMPER_5MM
- J2: value Fan_conn -> Encoder and LCD interface; footprint Pin_Headers:Pin_Header_Straight_1x04_Pitch2.54mm -> Pin_Headers:Pin_Header_Straight_1x07_Pitch2.54mm
- J9: value GPIO -> Load_on_switch
- Q4: footprint Load_mosfet -> LoadResistor:Load_mosfet
- R13: value 0.1 -> 10K; footprint Loadresistor -> Resistors_SMD:R_0805_HandSoldering
- R17: value 20K -> 100R
- R18: value 1M -> 20K; moved to F.Cu
- R22: value 10K -> 1M; moved to B.Cu
- R23: value 20K -> 10K; moved to F.Cu
- R24: value 2K -> 20K; moved to F.Cu
- R27: value 1K -> 2K; moved to B.Cu
- R29: value R -> 1K
- R30: value 100R -> R
- R31: value 0R1 -> 100R; footprint Resistors_SMD:R_1206_HandSoldering -> Resistors_SMD:R_0805_HandSoldering; moved to F.Cu
- R32: value 20K -> 0R1; footprint Resistors_SMD:R_0805_HandSoldering -> Resistors_SMD:R_1206_HandSoldering; moved to F.Cu
- R33: value 100K -> 20K; moved to F.Cu
- R34: value 1K6 -> 100K
- R35, R37: value 2k7 -> 1K6
- R38: value 1K6 -> 2k7
- R5: value R -> 2K2
- R7: value 2M2 -> 1M8
- RV3: value POT_TRIM -> 5K
- RV4: value POT_TRIM -> 10K
- U10: value Temp amp -> MCP4725; footprint TO_SOT_Packages_SMD:SOT-23-5 -> TO_SOT_Packages_SMD:TSOT-23-6_HandSoldering
- U11: value LM35 -> AD8628; footprint TO_SOT_Packages_THT:TO-220-3_Vertical -> Housings_SOIC:SOIC-8_3.9x4.9mm_Pitch1.27mm
- U12: value Bluepill -> Temp amp; footprint Libs:Bluepill -> TO_SOT_Packages_SMD:SOT-23-5
- U13: value DS3231 RTC -> LM35; footprint Housings_SOIC:SOIC-16W_7.5x10.3mm_Pitch1.27mm -> TO_SOT_Packages_THT:TO-220-3_Vertical
- U14: value TRIG -> DS3231 RTC; footprint TO_SOT_Packages_SMD:SOT-23-6_Handsoldering -> Housings_SOIC:SOIC-16W_7.5x10.3mm_Pitch1.27mm
- U15: value SN74LVC2G14 -> Bluepill; footprint TO_SOT_Packages_SMD:SOT-23-6_Handsoldering -> Libs:Bluepill
- U16: value PC817 -> TRIG; footprint Housings_DIP:DIP-4_W7.62mm -> TO_SOT_Packages_SMD:SOT-23-6_Handsoldering
- U17: value LT1054 neg5v -> SN74LVC2G14; footprint Housings_DIP:DIP-8_W7.62mm_LongPads -> TO_SOT_Packages_SMD:SOT-23-6_Handsoldering
- U18: value INA219 -> PC817; footprint TO_SOT_Packages_SMD:SOT-23-8_Handsoldering -> Housings_DIP:DIP-4_W7.62mm; moved to F.Cu
- U19: value LM7805 -> LT1054 neg5v; footprint TO_SOT_Packages_THT:TO-220-3_Vertical -> Housings_DIP:DIP-8_W7.62mm_LongPads
- U20: value LM1117-3.3 -> INA219; footprint TO_SOT_Packages_SMD:SOT-223-3_TabPin2 -> TO_SOT_Packages_SMD:SOT-23-8_Handsoldering
- U21: value Vref -> LM1117-3.3; footprint Housings_SOIC:SOIC-8_3.9x4.9mm_Pitch1.27mm -> TO_SOT_Packages_SMD:SOT-223-3_TabPin2
- U22: value AD8628 -> LM7805; footprint Housings_SOIC:SOIC-8_3.9x4.9mm_Pitch1.27mm -> TO_SOT_Packages_THT:TO-220-3_Vertical; moved to F.Cu
- U6: value Current amp -> AD5245; footprint Housings_DIP:DIP-8_W7.62mm_Socket_LongPads -> TO_SOT_Packages_SMD:SOT-23-8_Handsoldering; moved to B.Cu
- U7: value Volt sense -> Current amp
- U8: value MCP4725 -> AD5245; footprint TO_SOT_Packages_SMD:TSOT-23-6_HandSoldering -> TO_SOT_Packages_SMD:SOT-23-8_Handsoldering; moved to B.Cu
- U9: value AD8628 -> Volt sense; footprint Housings_SOIC:SOIC-8_3.9x4.9mm_Pitch1.27mm -> Housings_DIP:DIP-8_W7.62mm_Socket_LongPads; moved to F.Cu
- moved R36 502.2 mm to (433.4, -1.95)
- moved R37 492.2 mm to (428.1, 4.00)
- moved D7 487.3 mm to (410.8, 25.5)
- moved D6 483.3 mm to (415.3, 31.0)
- moved R34 482.4 mm to (410.7, 19.6)
- moved D8 479.4 mm to (423.2, 9.95)
- moved D9 474.5 mm to (417.7, 15.8)
- moved R35 469.1 mm to (417.7, 9.95)
- moved D5 462.2 mm to (399.7, 36.8)
- moved R38 449.2 mm to (399.7, 30.9)
- moved J14 330.1 mm to (-91.6, 114.9), turned to 0 degrees
- moved U17 317.2 mm to (-92.3, 121.2), turned to 0 degrees
- moved U18 298.7 mm to (-69.3, 96.2), turned to 0 degrees
- moved C1 298.3 mm to (199.6, 137.7), turned to 270 degrees
- moved R31 293.6 mm to (-57.9, 107.4), turned to 0 degrees
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Connections:
- C10 pad 1: +12V -> Net-(C10-Pad1)
- C11 pad 2: Earth -> Net-(C11-Pad2)
- C12 pad 1: Net-(C12-Pad1) -> +5V
- C12 pad 2: Net-(C12-Pad2) -> Earth
- C33 pad 1: +12V -> +5V
- C35 pad 1: +12V -> Net-(C35-Pad1)
- C36 pad 1: +5V -> +3V3
- C37 pad 1: +12V -> +5V
- C38 pad 1: Net-(C38-Pad1) -> +12V
- C39 pad 1: Net-(C39-Pad1) -> +12V
- C40 pad 1: +3V3 -> +12V
- C41 pad 1: +5V -> Net-(C41-Pad1)
- C8 pad 1: +5V -> +12V
- D6 pad 2: +5V -> Net-(D6-Pad2)
- D7 pad 2: +12V -> +5V
- D8 pad 1: -5V -> Net-(D8-Pad1)
- D8 pad 2: Net-(D8-Pad2) -> +12V
- D9 pad 1: Net-(D9-Pad1) -> -5V
- J1 pad 2: encB -> +12V
- J1 pad 3: encA -> fan_tach
- J1 pad 4: encBTN -> fan_PWM
- J10 pad 1: (no net) -> Net-(J10-Pad1)
- J10 pad 2: Earth -> Net-(J10-Pad2)
- J11 pad 1: trig -> Net-(J11-Pad1)
- J11 pad 2: Net-(J11-Pad2) -> Earth
- J12 pad 1: Net-(J12-Pad1) -> trig
- J12 pad 2: +3V3 -> Net-(J12-Pad2)
- J13 pad 2: Net-(D4-Pad1) -> +3V3
- J14 pad 1: Net-(C24-Pad1) -> Net-(J14-Pad1)
- J14 pad 2: Earth -> Net-(D4-Pad1)
- J2 pad 2: +12V -> encB
- J2 pad 3: (no net) -> encA
- J2 pad 4: fan_PWM -> encBTN
- J9 pad 1: Net-(J9-Pad1) -> Earth
- L2 pad 1: Net-(C39-Pad1) -> Net-(C35-Pad1)
- R10 pad 2: Net-(C12-Pad1) -> Net-(C11-Pad1)
- R11 pad 2: Net-(C11-Pad1) -> Net-(C10-Pad1)
- R12 pad 1: Net-(Q4-Pad1) -> Net-(R12-Pad1)
- R12 pad 2: Earth -> Net-(Q4-Pad2)
- R13 pad 1: Net-(Q4-Pad2) -> Net-(Q4-Pad1)
- R17 pad 1: Earth -> Curr
- R18 pad 1: Net-(R16-Pad1) -> Earth
- R18 pad 2: Earth -> Net-(R18-Pad2)
- R19 pad 1: Earth -> Net-(R16-Pad1)
- R19 pad 2: Net-(R17-Pad2) -> Earth
- R20 pad 1: Net-(J8-Pad1) -> Earth
- R20 pad 2: Net-(R16-Pad1) -> Net-(R18-Pad2)
- R21 pad 1: Net-(J8-Pad2) -> Net-(J8-Pad1)
- R21 pad 2: Net-(R17-Pad2) -> Net-(R16-Pad1)
- R22 pad 1: Net-(R22-Pad1) -> Net-(J8-Pad2)
- R22 pad 2: Earth -> Net-(R18-Pad2)
- R23 pad 1: CurrentSet -> Net-(R23-Pad1)
- R23 pad 2: Net-(R23-Pad2) -> Earth
- R24 pad 1: CurrentSet -> Net-(R24-Pad1)
- R24 pad 2: Net-(R24-Pad2) -> LoadBlockTemp
- R25 pad 1: Net-(R25-Pad1) -> CurrentSet
- R25 pad 2: LoadBlockTemp -> Net-(R25-Pad2)
- R26 pad 2: Net-(R25-Pad1) -> Net-(R24-Pad1)
- R27 pad 1: +3V3 -> CurrentSet
- R27 pad 2: SDA -> Net-(R27-Pad2)
- R28 pad 2: SCL -> SDA
- R29 pad 1: Net-(J12-Pad1) -> +3V3
- R29 pad 2: Earth -> SCL
- R30 pad 1: Net-(D4-Pad2) -> Net-(J13-Pad1)
- R30 pad 2: Net-(J13-Pad1) -> Earth
- R31 pad 1: Net-(C27-Pad1) -> Net-(D4-Pad2)
- R31 pad 2: Net-(C24-Pad1) -> Net-(J14-Pad1)
- R32 pad 1: Net-(C31-Pad1) -> Net-(C27-Pad1)
- R32 pad 2: Net-(R32-Pad2) -> Net-(C24-Pad1)
- R33 pad 2: -5V -> Net-(R33-Pad2)
- R34 pad 1: Net-(D5-Pad1) -> Net-(C31-Pad1)
- R34 pad 2: Earth -> -5V
- R35 pad 1: Net-(D6-Pad1) -> Net-(D5-Pad1)
- R37 pad 1: Net-(D8-Pad2) -> Earth
- R37 pad 2: Earth -> Net-(D6-Pad1)
- R38 pad 1: Earth -> Net-(D8-Pad1)
- R38 pad 2: Net-(D9-Pad1) -> Earth
- R6 pad 1: Net-(Q4-Pad2) -> Net-(R12-Pad1)
- R8 pad 1: Net-(C12-Pad2) -> Net-(C11-Pad2)
- R8 pad 2: Net-(Q4-Pad2) -> Net-(R12-Pad1)
- R9 pad 1: Net-(C11-Pad1) -> Net-(C10-Pad1)
- RV3 pad 1: Net-(RV3-Pad1) -> Net-(R27-Pad2)
- RV3 pad 2: +5V -> Earth
- RV3 pad 3: Net-(RV3-Pad3) -> Earth
- RV4 pad 1: Net-(RV4-Pad1) -> Earth
- RV4 pad 2: +5V -> Net-(RV4-Pad2)
- TP2 pad 1: Net-(RV6-Pad3) -> Net-(RV4-Pad3)
- U10 pad 1: Net-(R25-Pad1) -> Net-(R23-Pad1)
- U10 pad 2: +5V -> Earth
- U10 pad 3: Net-(U10-Pad3) -> 4.096V
- U10 pad 4: LoadBlockTemp -> SDA
- U10 pad 5: Earth -> SCL
- U11 pad 1: +5V -> (no net)
- U11 pad 2: Earth -> Net-(R25-Pad2)
- U11 pad 3: Net-(U10-Pad3) -> Net-(R23-Pad1)
- U12 pad 1: (no net) -> Net-(R24-Pad1)
- U12 pad 2: (no net) -> +5V
- U12 pad 3: (no net) -> Net-(U12-Pad3)
- U12 pad 4: (no net) -> LoadBlockTemp
- U12 pad 5: Net-(J9-Pad2) -> Earth
- U13 pad 1: (no net) -> +5V
- U13 pad 2: +3V3 -> Earth
- U13 pad 3: (no net) -> Net-(U12-Pad3)
- U14 pad 1: trig -> (no net)
- U14 pad 2: Earth -> +3V3
- U14 pad 5: +3V3 -> Earth
- U14 pad 6: Net-(J11-Pad2) -> Earth
- U15 pad 2: Earth -> (no net)
- U15 pad 3: Net-(J12-Pad1) -> (no net)
- U15 pad 4: trig -> (no net)
- U15 pad 5: +3V3 -> Net-(J10-Pad2)
- U15 pad 6: (no net) -> Net-(J10-Pad1)
- U16 pad 1: Net-(D4-Pad2) -> trig
- U16 pad 2: Net-(D4-Pad1) -> Earth
- U16 pad 3: Net-(J12-Pad1) -> (no net)
- U16 pad 4: +3V3 -> (no net)
- U17 pad 1: Net-(C31-Pad1) -> (no net)
- U17 pad 2: Net-(C23-Pad1) -> Earth
- U17 pad 3: Earth -> Net-(J13-Pad1)
- U17 pad 4: Net-(C23-Pad2) -> trig
- U17 pad 5: -5V -> +3V3
- U17 pad 6: Net-(R32-Pad2) -> (no net)
- U18 pad 1: Net-(C24-Pad1) -> Net-(D4-Pad2)
- U18 pad 2: Net-(C27-Pad1) -> Net-(D4-Pad1)
- U18 pad 3: Earth -> Net-(J13-Pad1)
- U19 pad 1: +12V -> Net-(C31-Pad1)
- U19 pad 2: Earth -> Net-(C23-Pad1)
- U19 pad 3: Net-(C39-Pad1) -> Earth
- U20 pad 1: Earth -> Net-(C24-Pad1)
- U20 pad 2: +3V3 -> Net-(C27-Pad1)
- U20 pad 3: +5V -> Earth
- U21 pad 1: (no net) -> Earth
- U21 pad 2: +12V -> +3V3
- U21 pad 3: Net-(C38-Pad1) -> +5V
- U22 pad 1: (no net) -> +12V
- U22 pad 2: 4.096V -> Earth
- U22 pad 3: Net-(RV6-Pad3) -> Net-(C35-Pad1)
- U23 pad 3: Net-(D9-Pad2) -> Net-(D6-Pad2)
- U23 pad 4: Net-(D9-Pad2) -> Net-(D6-Pad2)
- U3 pad 6: Net-(C11-Pad1) -> Net-(C10-Pad1)
- U4 pad 2: Net-(Q4-Pad2) -> Net-(R12-Pad1)
- U4 pad 6: Net-(C12-Pad1) -> Net-(C11-Pad1)
- U6 pad 1: Net-(RV3-Pad1) -> +5V
- U6 pad 2: Curr -> +5V
- U6 pad 3: Net-(R14-Pad2) -> Earth
- U6 pad 4: -5V -> SCL
- U6 pad 5: (no net) -> SDA
- U6 pad 6: Curr -> Earth
- U6 pad 7: +5V -> Net-(U6-Pad7)
- U6 pad 8: Net-(RV3-Pad3) -> Net-(U6-Pad8)
- U7 pad 1: Net-(RV4-Pad3) -> Net-(U6-Pad8)
- U7 pad 2: Net-(R16-Pad1) -> Net-(R17-Pad2)
- U7 pad 3: Net-(R17-Pad2) -> Net-(R14-Pad2)
- U7 pad 6: Net-(R15-Pad2) -> Net-(R17-Pad2)
- U7 pad 8: Net-(RV4-Pad1) -> Net-(U6-Pad7)
- U8 pad 1: Net-(R22-Pad1) -> +5V
- U8 pad 2: Earth -> +5V
- U8 pad 3: 4.096V -> Earth
- U8 pad 4: SDA -> SCL
- U8 pad 5: SCL -> SDA
- U8 pad 6: Earth -> +5V
- U9 pad 1: (no net) -> Net-(U8-Pad8)
- U9 pad 2: Net-(R23-Pad2) -> Net-(R18-Pad2)
- U9 pad 3: Net-(R22-Pad1) -> Net-(R16-Pad1)
- U9 pad 4: Earth -> -5V
- U9 pad 6: Net-(R23-Pad2) -> Net-(R15-Pad2)
- U9 pad 8: (no net) -> Net-(U8-Pad7)
Routing:
- net -5V: track 259.8 -> 8.73 mm
- net +12V: track 276.9 -> 34.0 mm, vias 1 -> 0
- net SCL: track 198.4 -> 26.5 mm, vias 1 -> 0
- net +5V: track 272.2 -> 106.9 mm
- net SDA: track 192.8 -> 28.5 mm, vias 1 -> 0
- net Earth: track 188.2 -> 74.6 mm
- net +3V3: track 76.0 -> 0.00 mm, vias 2 -> 0
- net Net-(R12-Pad1): track 0.00 -> 42.2 mm
- net Net-(Q4-Pad2): track 46.1 -> 13.0 mm
- net Net-(C24-Pad1): track 24.7 -> 0.00 mm
- net Net-(RV6-Pad3): track 21.3 -> 0.00 mm, vias 1 -> 0
- net Net-(C31-Pad1): track 19.1 -> 0.00 mm
- net Net-(C27-Pad1): track 18.8 -> 0.00 mm
- net Net-(C10-Pad1): track 0.00 -> 18.5 mm
- net Net-(R25-Pad2): track 0.00 -> 18.3 mm
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Other:
- net class power: clearance 0.4 -> 0.25

Commit message: v2 done
Parts:
- removed the C42 at (144.3, 135.6)
- removed D1, D2: D_ALT, Diodes_SMD:D_MELF-RM10_Universal_Handsoldering
- removed D5, D6, D7, D8, D9: LED, LEDs:LED_0805_HandSoldering
- removed J4, J5: OUT2, Pin_Headers:Pin_Header_Straight_1x02_Pitch2.54mm
- removed Q1, Q2: BC847, TO_SOT_Packages_SMD:SOT-23_Handsoldering
- removed Q3: IRF7341, Housings_SOIC:SOIC-8_3.9x4.9mm_Pitch1.27mm
- removed R1, R2: 100R, Resistors_SMD:R_0805_HandSoldering
- removed R28, R29: 1K, Resistors_SMD:R_0805_HandSoldering
- removed R3, R4: 10K, Resistors_SMD:R_0805_HandSoldering
- removed R35, R37: 1K6, Resistors_SMD:R_0805_HandSoldering
- removed R36, R38, R39: 2k7, Resistors_SMD:R_0805_HandSoldering
- removed U17: SN74LVC2G14, TO_SOT_Packages_SMD:SOT-23-6_Handsoldering
- removed U23: LM321, TO_SOT_Packages_SMD:SOT-23-5
- added BT1: Battery_Cell, Libs:JUMPER_5MM, F.Cu at (175.0, 80.3)
- added C14: 0.1u, Capacitors_SMD:C_0805_HandSoldering, B.Cu at (182.9, 109.2)
- added REF**: MountingHole_3.2mm_M3, Mounting_Holes:MountingHole_3.2mm_M3, F.Cu at (197.9, 119.1)
- added REF**: MountingHole_3.2mm_M3, Mounting_Holes:MountingHole_3.2mm_M3, F.Cu at (223.8, 88.6)
- added REF**: MountingHole_3.2mm_M3, Mounting_Holes:MountingHole_3.2mm_M3, F.Cu at (177.3, 51.8)
- added REF**: MountingHole_3.2mm_M3, Mounting_Holes:MountingHole_3.2mm_M3, F.Cu at (137.9, 91.7)
- C17: renamed from C16; moved to F.Cu
- C2, C4, L2, R31, R33, R34, U14, U21: moved to B.Cu
- C21: renamed from C20; moved to B.Cu
- C22: renamed from C21; moved to B.Cu
- C23: renamed from C22; moved to B.Cu
- C25: renamed from C24; moved to B.Cu
- C26: renamed from C25; moved to B.Cu
- C30: renamed from C29; moved to B.Cu
- C34: renamed from C33; moved to B.Cu
- C37: renamed from C36; moved to B.Cu
- C38: renamed from C37; moved to B.Cu
- moved J2 294.7 mm to (167.6, 50.5), turned to 270 degrees
- moved BT1 284.3 mm to (191.3, 75.9)
- moved J3 267.3 mm to (144.0, 86.9), turned to 180 degrees
- moved C20 265.9 mm to (135.6, 144.8)
- moved C22 264.8 mm to (172.2, 50.8), turned to 90 degrees
- moved J1 264.6 mm to (144.3, 101.1), turned to 180 degrees
- moved J9 261.4 mm to (179.6, 60.2), turned to 270 degrees
- moved U14 259.2 mm to (180.3, 68.3), turned to 270 degrees
- moved C21 257.5 mm to (191.0, 66.0)
- moved U16 249.7 mm to (144.0, 67.3), turned to 180 degrees
- moved C3 249.3 mm to (138.2, 106.7), turned to 270 degrees
- moved C32 245.8 mm to (190.8, 62.5)
- moved C7 244.1 mm to (150.1, 122.4), turned to 180 degrees
- moved C2 241.9 mm to (147.3, 56.4), turned to 270 degrees
- moved J11 241.3 mm to (144.5, 106.4)
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- renumbered C9 to C12, C12 to C13, C13 to C14, C14 to C15, C15 to C16, C17 to C18, C18 to C19, C19 to C20, C23 to C24, C26 to C27, C27 to C28, C28 to C29, C30 to C31, C31 to C32, C32 to C33, C34 to C35, C35 to C36, C38 to C39, C39 to C40, C40 to C41, C41 to C42, C43 to C8, C8 to C9, R26 to R25, R25 to R26, U9 to U8, U8 to U9
Connections:
- U15 pad 25: out1 -> (no net)
- U15 pad 26: out2 -> (no net)
- U16 pad 3: (no net) -> Net-(J13-Pad1)
- U16 pad 4: (no net) -> trig
Routing:
- net Earth: track 74.6 -> 880.0 mm, vias 0 -> 1
- net +5V: track 106.9 -> 488.7 mm, vias 0 -> 2
- net SDA: track 28.5 -> 343.1 mm, vias 0 -> 3
- net SCL: track 26.5 -> 305.3 mm, vias 0 -> 2
- net -5V: track 8.73 -> 250.4 mm
- net +12V: track 34.0 -> 253.7 mm, vias 0 -> 2
- net +3V3: track 0.00 -> 201.7 mm, vias 0 -> 3
- net OverTemp: track 0.00 -> 117.5 mm, vias 0 -> 2
- net comperator: track 0.00 -> 69.4 mm, vias 0 -> 1
- net LoadBlockTemp: track 0.00 -> 68.9 mm, vias 0 -> 1
- net trig: track 0.00 -> 47.8 mm, vias 0 -> 1
- net fan_tach: track 0.00 -> 46.5 mm
- net encBTN: track 0.00 -> 37.1 mm
- net encA: track 0.00 -> 34.4 mm
- net encB: track 0.00 -> 30.1 mm
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Other:
- board size 97 x 99.8 mm -> 97 x 100.1 mm

Commit message: press "b"
Routing:
- net (no net): track 7.70 -> 0.78 mm
Changed lines of the file:
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@@
 (kicad_pcb (version 4) (host pcbnew 4.0.7)
   (general
-    (links 0)
+    (links 298)
     (no_connects 6)
-    (area 131.245 30.828001 249.864286 147.655)
+    (area 128.314857 30.828001 249.864286 147.655)
     (thickness 1.6)
     (drawings 6)
-    (tracks 1134)
+    (tracks 1132)
     (zones 0)
     (modules 126)
@@
     (0 F.Cu signal)
     (31 B.Cu signal)
-    (32 B.Adhes user hide)
-    (33 F.Adhes user hide)
+    (32 B.Adhes user)
+    (33 F.Adhes user)
     (34 B.Paste user hide)
     (35 F.Paste user hide)
     (36 B.SilkS user hide)
     (37 F.SilkS user hide)
-    (38 B.Mask user hide)
-    (39 F.Mask user hide)
+    (38 B.Mask user)
+    (39 F.Mask user)
     (40 Dwgs.User user hide)
     (41 Cmts.User user hide)
     (42 Eco1.User user hide)
     (43 Eco2.User user hide)
-    (44 Edge.Cuts user)
+    (44 Edge.Cuts user hide)
     (45 Margin user hide)
     (46 B.CrtYd user)
@@
   (gr_line (start 228.854 146.05) (end 229.108 45.974) (layer Edge.Cuts) (width 0.15))
   (segment (start 167.778 94.488) (end 168.556 94.488) (width 0.4) (layer B.Cu) (net 0) (status 30))
-  (segment (start 174.01 58.928) (end 180.212 58.928) (width 0.4) (layer B.Cu) (net 0))
-  (segment (start 180.212 58.928) (end 180.721 59.437) (width 0.4) (layer B.Cu) (net 0))
   (segment (start 187.198 76.962) (end 181.271 76.962) (width 0.4) (layer B.Cu) (net 1))
   (segment (start 181.271 76.962) (end 178.435 74.126) (width 0.4) (layer B.Cu) (net 1))

Commit message: Before starting saturday
Parts:
- added R28, R29: 1K, Resistors_SMD:R_0805_HandSoldering, F.Cu at (180.6, 156.1)
Connections:
- BT1 pad 1: Earth -> Net-(BT1-Pad1)
- U14 pad 1: (no net) -> Net-(U14-Pad1)
- U14 pad 3: (no net) -> Net-(U14-Pad3)
- U14 pad 4: (no net) -> Net-(U14-Pad4)
- U15 pad 1: (no net) -> Net-(U15-Pad1)
- U15 pad 2: (no net) -> Net-(U15-Pad2)
- U15 pad 21: (no net) -> Net-(U15-Pad21)
- U15 pad 22: (no net) -> Net-(U15-Pad22)
- U15 pad 23: (no net) -> Net-(U15-Pad23)
- U15 pad 24: (no net) -> Net-(U15-Pad24)
- U15 pad 25: (no net) -> out1
- U15 pad 26: (no net) -> out2
- U15 pad 28: (no net) -> Net-(U15-Pad28)
- U15 pad 29: (no net) -> Net-(U15-Pad29)
- U15 pad 3: (no net) -> Net-(U15-Pad3)
- U15 pad 37: (no net) -> Net-(U15-Pad37)
- U15 pad 38: (no net) -> Net-(U15-Pad38)
- U15 pad 4: (no net) -> Net-(U15-Pad4)
- U15 pad 7: (no net) -> Net-(U15-Pad7)
- U15 pad 8: (no net) -> Net-(U15-Pad8)
- U19 pad 7: (no net) -> Net-(U19-Pad7)
- U24 pad 1: (no net) -> Net-(U24-Pad1)
- U24 pad 7: (no net) -> Net-(U24-Pad7)
- U24 pad 8: (no net) -> Net-(U24-Pad8)
- U3 pad 1: (no net) -> Net-(U3-Pad1)
- U4 pad 5: (no net) -> Net-(U4-Pad5)
- U5 pad 1: (no net) -> Net-(U5-Pad1)
- U5 pad 5: (no net) -> Net-(U5-Pad5)
- U5 pad 8: (no net) -> Net-(U5-Pad8)
- U7 pad 5: (no net) -> Net-(U7-Pad5)
- U8 pad 5: (no net) -> Net-(U8-Pad5)
Routing:
- net out1: track 0.00 -> 0.78 mm
- net (no net): track 0.78 -> 0.00 mm
