File: HW/v2/file5AD8A8B3.sch (KiCad schematic (older format))
At the start: 33 parts, among them J15 Barrel_Jack, U19 LT1054 neg5v, U20 INA219, U21 LM1117-3.3, U22 LM7805, U24 Vref, U25 AD8628

Commit message: Before starting saturday
Parts:
- U21: symbol LM1117-3.3 -> LM1117-3.3-RESCUE-v2
Changed lines of the file:
@@
 EESchema Schematic File Version 2
+LIBS:v2-rescue
 LIBS:power
 LIBS:device
@@
 LIBS:contrib
 LIBS:valves
-LIBS:Peters
-LIBS:BLUEPILL
 LIBS:v2-cache
 EELAYER 25 0
@@
 $EndComp
 $Comp
-L LM1117-3.3 U21
+L LM1117-3.3-RESCUE-v2 U21
 U 1 1 5ADAB666
 P 5400 2400
+AR Path="/5ADAB666" Ref="U21"  Part="1"
+AR Path="/5AD8A8B3/5ADAB666" Ref="U21"  Part="1"
 F 0 "U21" H 5250 2525 50  0000 C CNN
 F 1 "LM1117-3.3" H 5400 2525 50  0000 L CNN
