File: HW/v2/MCU.sch (KiCad schematic (older format))
At the start: 19 parts, among them J10 GPIO, J11 RST, J12 ScopeTest, J13 Trigger BTN, J14 External trigger, J9 Load_on_switch, U14 DS3231 RTC, U15 Bluepill, U16 TRIG, U18 PC817

Commit message: more
Parts:
- BT1: symbol Battery_Cell -> device:Battery_Cell
- C21, C22, C23: symbol C -> device:C
- D4: symbol 1N4148 -> Peters:1N4148
- J10, J11, J12, J13, J14, J9: symbol Conn_01x02 -> conn:Conn_01x02
- R28, R29: symbol R_Small -> device:R_Small
- R30, R31: symbol R -> device:R
- U14: symbol DS3231 -> Peters:DS3231
- U15: symbol Bluepill -> Peters:Bluepill
- U16: symbol SN74LVC2G14 -> Peters:SN74LVC2G14
- U18: symbol PC817 -> opto:PC817
Changed lines of the file:
@@
-EESchema Schematic File Version 2
-LIBS:power
-LIBS:device
-LIBS:switches
-LIBS:relays
-LIBS:motors
-LIBS:transistors
-LIBS:conn
-LIBS:linear
-LIBS:regul
-LIBS:74xx
-LIBS:cmos4000
-LIBS:adc-dac
-LIBS:memory
-LIBS:xilinx
-LIBS:microcontrollers
-LIBS:dsp
-LIBS:microchip
-LIBS:analog_switches
-LIBS:motorola
-LIBS:texas
-LIBS:intel
-LIBS:audio
-LIBS:interface
-LIBS:digital-audio
-LIBS:philips
-LIBS:display
-LIBS:cypress
-LIBS:siliconi
-LIBS:opto
-LIBS:atmel
-LIBS:contrib
-LIBS:valves
-LIBS:Peters
-LIBS:BLUEPILL
+EESchema Schematic File Version 4
 LIBS:v2-cache
-EELAYER 25 0
+EELAYER 26 0
 EELAYER END
 $Descr A4 11693 8268
@@
 SDA
 $Comp
-L R_Small R28
+L device:R_Small R28
 U 1 1 5ADB7193
 P 5250 2600
@@
 $EndComp
 $Comp
-L R_Small R29
+L device:R_Small R29
 U 1 1 5ADB719A
 P 5500 2600
@@
 $EndComp
 $Comp
-L +3.3V #PWR087
+L power:+3.3V #PWR087
 U 1 1 5ADB71A1
 P 5250 2450
@@
 $EndComp
 $Comp
-L +3.3V #PWR088
+L power:+3.3V #PWR088
 U 1 1 5ADB71A7
 P 5500 2450
@@
 $EndComp
 $Comp
-L GND #PWR089
+L power:GND #PWR089
 U 1 1 5ADB71AD
 P 1800 3050
@@
 OverTemp
 $Comp
-L GND #PWR090
+L power:GND #PWR090
 U 1 1 5ADB71BF
 P 5200 1650
@@
 LoadBlockTemp
 $Comp
-L Bluepill U15
+L Peters:Bluepill U15
 U 1 1 5ADB71CF
 P 2950 1800
@@
 $EndComp
 $Comp
-L Conn_01x02 J11
+L conn:Conn_01x02 J11
 U 1 1 5ADB71D6
 P 5400 1550
@@
 $EndComp
 $Comp
-L GND #PWR091
+L power:GND #PWR091
 U 1 1 5ADB71DD
 P 4200 1250
@@
 $EndComp
 $Comp
-L GND #PWR092
+L power:GND #PWR092
 U 1 1 5ADB71E3
 P 4200 1350
@@
 	4600 1450 4600 1400
 $Comp
-L +3.3V #PWR093
+L power:+3.3V #PWR093
 U 1 1 5ADB71EB
 P 4600 1400
@@
 	4950 2450 4950 2400
 $Comp
-L GND #PWR094
+L power:GND #PWR094
 U 1 1 5ADB71F3
 P 4950 2800
@@
 $EndComp
 $Comp
-L C C23
+L device:C C23
 U 1 1 5ADB71F9
 P 4950 2600
@@
 $EndComp
 $Comp
-L +3.3V #PWR095
+L power:+3.3V #PWR095
 U 1 1 5ADB7200
 P 4950 2400
@@
 	4700 2450 4700 2400
 $Comp
-L GND #PWR096
+L power:GND #PWR096
 U 1 1 5ADB7208
 P 4700 2800
@@
 $EndComp
 $Comp
-L C C22
+L device:C C22
 U 1 1 5ADB720E
 P 4700 2600
@@
 $EndComp
 $Comp
-L +3.3V #PWR097
+L power:+3.3V #PWR097
 U 1 1 5ADB7215
 P 4700 2400
@@
 $EndComp
 $Comp
-L +3.3V #PWR098
+L power:+3.3V #PWR098
 U 1 1 5ADB721B
 P 1500 3150
@@
 fan_PWM
 $Comp
-L Conn_01x02 J10
+L conn:Conn_01x02 J10
 U 1 1 5ADB7229
 P 4400 2650
@@
 $EndComp
 $Comp
-L PC817 U18
+L opto:PC817 U18
 U 1 1 5ADB8458
 P 9300 1350
@@
 $EndComp
 $Comp
-L 1N4148 D4
+L Peters:1N4148 D4
 U 1 1 5ADB845F
 P 9500 1400
@@
 $EndComp
 $Comp
-L R R31
+L device:R R31
 U 1 1 5ADB8466
 P 10250 1450
@@
 $EndComp
 $Comp
-L Conn_01x02 J14
+L conn:Conn_01x02 J14
 U 1 1 5ADB846D
 P 10150 2050
@@
 $EndComp
 $Comp
-L R R30
+L device:R R30
 U 1 1 5ADB8474
 P 9000 1800
@@
 $EndComp
 $Comp
-L GND #PWR099
+L power:GND #PWR099
 U 1 1 5ADB847B
 P 9000 2100
@@
 trig
 $Comp
-L Conn_01x02 J12
+L conn:Conn_01x02 J12
 U 1 1 5ADB8482
 P 6300 1600
@@
 $EndComp
 $Comp
-L Conn_01x02 J13
+L conn:Conn_01x02 J13
 U 1 1 5ADB8489
 P 8450 1100
@@
 $EndComp
 $Comp
-L GND #PWR0100
+L power:GND #PWR0100
 U 1 1 5ADB8490
 P 8350 1950
@@
 $EndComp
 $Comp
-L GND #PWR0101
+L power:GND #PWR0101
 U 1 1 5ADB8496
 P 7400 1700
@@
 $EndComp
 $Comp
-L +3.3V #PWR0102
+L power:+3.3V #PWR0102
 U 1 1 5ADB849C
 P 7400 1300
@@
 $EndComp
 $Comp
-L +3.3V #PWR0103
+L power:+3.3V #PWR0103
 U 1 1 5ADB84A2
 P 8350 1550
@@
 $EndComp
 $Comp
-L +3.3V #PWR0104
+L power:+3.3V #PWR0104
 U 1 1 5ADB84A8
 P 8650 1000
@@
 $EndComp
 $Comp
-L +3.3V #PWR0105
+L power:+3.3V #PWR0105
 U 1 1 5ADB84AE
 P 8950 1150
@@
 	9950 1600 9650 1600
 $Comp
-L SN74LVC2G14 U16
+L Peters:SN74LVC2G14 U16
 U 1 1 5ADB84D4
 P 7400 1550
@@
 $EndComp
 $Comp
-L SN74LVC2G14 U16
+L Peters:SN74LVC2G14 U16
 U 2 1 5ADB84DB
 P 8350 1800
@@
 Trigger
 $Comp
-L Battery_Cell BT1
+L device:Battery_Cell BT1
 U 1 1 5ADB8A71
 P 2750 4400
@@
 $EndComp
 $Comp
-L GND #PWR0106
+L power:GND #PWR0106
 U 1 1 5ADB8A78
 P 2750 4550
@@
 $EndComp
 $Comp
-L DS3231 U14
+L Peters:DS3231 U14
 U 1 1 5ADB8A7E
 P 2200 4600
@@
 SDA
 $Comp
-L +3.3V #PWR0107
+L power:+3.3V #PWR0107
 U 1 1 5ADB8A87
 P 1350 4100
@@
 $EndComp
 $Comp
-L C C21
+L device:C C21
 U 1 1 5ADB8A8D
 P 1350 4250
@@
 $EndComp
 $Comp
-L GND #PWR0108
+L power:GND #PWR0108
 U 1 1 5ADB8A94
 P 1350 4450
@@
 	2750 4200 2550 4200
 $Comp
-L Conn_01x02 J9
+L conn:Conn_01x02 J9
 U 1 1 5ADC9E0D
 P 950 2850
@@
 $EndComp
 $Comp
-L GND #PWR0109
+L power:GND #PWR0109
 U 1 1 5ADC9FA5
 P 1150 3000
