File: HW/v2/file5AD8A8C6.sch (KiCad schematic (older format))
At the start: 62 parts, among them J6 DUT+, J7 DUT-, J8 Remote_sense, Q4 STW45NM50, U10 MCP4725, U11 AD8628, U12 Temp amp, U13 LM35, U2 TL431A, U3 ADS1115, U4 Gate DRV, U5 Volt buffer, U6 AD5245, U7 Current amp, U8 Volt sense, U9 AD5245

Commit message: more
Parts:
- removed U5: Volt buffer, Housings_DIP:DIP-8_W7.62mm_Socket_LongPads, symbol OP07
- C10, C11, C13, C14, C15, C16, C17, C18, C19, C20, C5, C6, C7, C8, C9: symbol C -> device:C
- C12: symbol CP1 -> device:CP1
- D3: symbol D_Schottky -> device:D_Schottky
- F1: symbol Fuse -> device:Fuse
- J6, J7: symbol Conn_01x01 -> conn:Conn_01x01
- J8: symbol Conn_01x02 -> conn:Conn_01x02
- Q4: symbol STW45NM50 -> Peters:STW45NM50
- R-shunt1, R10, R11, R12, R13, R14, R15, R16, R17, R18, R19, R20, R21, R22, R23, R24, R25, R26, R27, R5, R6, R7, R8, R9: symbol R -> device:R
- U10: symbol MCP4725 -> Peters:MCP4725
- U11: symbol AD8628 -> Peters:AD8628
- U12: symbol LM321 -> linear:LM321
- U13: symbol LM35 -> Peters:LM35
- U2: symbol TL431A -> Peters:TL431A
- U3: symbol ADS1115 -> Peters:ADS1115
- U4, U7, U8: symbol OP07 -> linear:OP07
- U6, U9: symbol AD5245 -> Peters:AD5245
Connections:
- net +5V: now also U12.5 (V+); no longer U12.2 (V-)
- net Earth: now also U12.2 (V-); no longer U12.5 (V+)
- net at R11.1: now also R15.2, R16.2, U8.6
- net at U13.3 (Out): now also U12.1 (+); no longer U12.3 (-)
- net at R24.1, R25.2: now also U12.3 (-); no longer U12.1 (+)
- no-connect marks 2 -> 0
